File: project_kicad/strange_games.kicad_sch (KiCad schematic)
At the start: 123 parts, among them J1 Display, M1 Motor_DC, Q1 Si2302A, Q2 Q_Photo, Q3 Si2302A, Q4 Q_Photo, SW1 SW_Push, SW10 SW_Push, SW11 SW_Push, SW12 SW_Push, SW4 SW_Push, SW5 SW_Push, SW6 SW_Push, SW7 SW_Push, SW8 SW_Push, SW9 SW_Push, U1 charge controller, U2 boost converter, U3 LDL1117S33R, U4 ESP32-DEVKIT-V1, U5 TMP112xxDRL, U6 vibrating_sensor, U7 LSM6DS3, U8 MQ-135 gas sensor

Commit message: updated placements for pcb
Parts:
- L1, M1: footprint (none) -> Connector_PinHeader_2.54mm:PinHeader_1x02_P2.54mm_Vertical
- Q2, Q4: footprint (none) -> LED_THT:LED_D4.0mm
- U1: footprint Library:charge_controller_module_tp4056 -> SnapEDA Library:charge_controller_module_tp4056
- U2: footprint Library:CKCS BS-01 MT-3608 Boost Converter -> SnapEDA Library:CKCS BS-01 MT-3608 Boost Converter
- U6: footprint (none) -> Connector_PinHeader_2.54mm:PinHeader_1x03_P2.54mm_Vertical
Changed lines of the file:
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@@
       (effects (font (size 1.27 1.27)) (justify left) hide)
     )
-    (property "Footprint" "" (at 130.81 22.86 0)
+    (property "Footprint" "LED_THT:LED_D4.0mm" (at 130.81 22.86 0)
       (effects (font (size 1.27 1.27)) hide)
     )
@@
       (effects (font (size 1.27 1.27)) (justify left) hide)
     )
-    (property "Footprint" "" (at 114.3 22.86 0)
+    (property "Footprint" "LED_THT:LED_D4.0mm" (at 114.3 22.86 0)
       (effects (font (size 1.27 1.27)) hide)
     )
@@
       (effects (font (size 1.27 1.27)) (justify left))
     )
-    (property "Footprint" "" (at 109.22 171.45 0)
+    (property "Footprint" "Connector_PinHeader_2.54mm:PinHeader_1x02_P2.54mm_Vertical" (at 109.22 171.45 0)
       (effects (font (size 1.27 1.27)) hide)
     )
@@
       (effects (font (size 1.27 1.27)) (justify left))
     )
-    (property "Footprint" "" (at 115.57 202.946 0)
+    (property "Footprint" "Connector_PinHeader_2.54mm:PinHeader_1x02_P2.54mm_Vertical" (at 115.57 202.946 0)
       (effects (font (size 1.27 1.27)) hide)
     )
@@
       (effects (font (size 1.27 1.27)))
     )
-    (property "Footprint" "Library:charge_controller_module_tp4056" (at 40.64 177.8 0)
+    (property "Footprint" "SnapEDA Library:charge_controller_module_tp4056" (at 40.64 177.8 0)
       (effects (font (size 1.27 1.27)) hide)
     )
@@
       (effects (font (size 1.27 1.27)))
     )
-    (property "Footprint" "" (at 149.86 10.16 0)
+    (property "Footprint" "Connector_PinHeader_2.54mm:PinHeader_1x03_P2.54mm_Vertical" (at 149.86 10.16 0)
       (effects (font (size 1.27 1.27)) hide)
     )
@@
       (effects (font (size 1.27 1.27)))
     )
-    (property "Footprint" "Library:CKCS BS-01 MT-3608 Boost Converter" (at 52.07 190.5 0)
+    (property "Footprint" "SnapEDA Library:CKCS BS-01 MT-3608 Boost Converter" (at 52.07 190.5 0)
       (effects (font (size 1.27 1.27)) hide)
     )
