File: project_kicad/strange_games.kicad_sch (KiCad schematic)
At the start: 93 parts, among them J1 Display, M1 Motor_DC, Q1 Si2302A, Q3 Si2302A, Q4 Q_Photo, SW1 SW_Push, SW10 SW_Push, SW11 SW_Push, SW2 SW_Push, SW3 SW_Push, SW4 SW_Push, SW5 SW_Push, SW6 SW_Push, SW7 SW_Push, SW8 SW_Push, SW9 SW_Push, U1 charge controller, U2 boost converter, U3 LDL1117S33R, U4 ESP32-DEVKIT-V1, U5 TMP112xxDRL, U6 vibrating_sensor, U7 LSM6DS3, U8 MQ-135 gas sensor

Commit message: kicad changes + trash esp32
made via's better to make it possible to create
Parts:
- D10, D11, D12, D13, D5, D6, D7, D8, D9: footprint LED_THT:LED_D5.0mm-4_RGB -> Library:library
Changed lines of the file:
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@@
       (effects (font (size 1.27 1.27)))
     )
-    (property "Footprint" "LED_THT:LED_D5.0mm-4_RGB" (at 128.27 156.21 0)
+    (property "Footprint" "Library:library" (at 128.27 156.21 0)
       (effects (font (size 1.27 1.27)) (justify left top) hide)
     )
@@
       (effects (font (size 1.27 1.27)))
     )
-    (property "Footprint" "LED_THT:LED_D5.0mm-4_RGB" (at 128.27 133.35 0)
+    (property "Footprint" "Library:library" (at 128.27 133.35 0)
       (effects (font (size 1.27 1.27)) (justify left top) hide)
     )
@@
       (effects (font (size 1.27 1.27)))
     )
-    (property "Footprint" "LED_THT:LED_D5.0mm-4_RGB" (at 152.4 156.21 0)
+    (property "Footprint" "Library:library" (at 152.4 156.21 0)
       (effects (font (size 1.27 1.27)) (justify left top) hide)
     )
@@
       (effects (font (size 1.27 1.27)))
     )
-    (property "Footprint" "LED_THT:LED_D5.0mm-4_RGB" (at 176.53 144.78 0)
+    (property "Footprint" "Library:library" (at 176.53 144.78 0)
       (effects (font (size 1.27 1.27)) (justify left top) hide)
     )
@@
       (effects (font (size 1.27 1.27)))
     )
-    (property "Footprint" "LED_THT:LED_D5.0mm-4_RGB" (at 152.4 133.35 0)
+    (property "Footprint" "Library:library" (at 152.4 133.35 0)
       (effects (font (size 1.27 1.27)) (justify left top) hide)
     )
@@
       (effects (font (size 1.27 1.27)))
     )
-    (property "Footprint" "LED_THT:LED_D5.0mm-4_RGB" (at 152.4 144.78 0)
+    (property "Footprint" "Library:library" (at 152.4 144.78 0)
       (effects (font (size 1.27 1.27)) (justify left top) hide)
     )
@@
       (effects (font (size 1.27 1.27)))
     )
-    (property "Footprint" "LED_THT:LED_D5.0mm-4_RGB" (at 176.53 156.21 0)
+    (property "Footprint" "Library:library" (at 176.53 156.21 0)
       (effects (font (size 1.27 1.27)) (justify left top) hide)
     )
@@
       (effects (font (size 1.27 1.27)))
     )
-    (property "Footprint" "LED_THT:LED_D5.0mm-4_RGB" (at 128.27 144.78 0)
+    (property "Footprint" "Library:library" (at 128.27 144.78 0)
       (effects (font (size 1.27 1.27)) (justify left top) hide)
     )
@@
       (effects (font (size 1.27 1.27)))
     )
-    (property "Footprint" "LED_THT:LED_D5.0mm-4_RGB" (at 176.53 133.35 0)
+    (property "Footprint" "Library:library" (at 176.53 133.35 0)
       (effects (font (size 1.27 1.27)) (justify left top) hide)
     )

Commit message: It should be remastered with events
Connections:
- net Luminodiodes: no longer U4.12 (RX0)
- net Alert: now reaches U5.3 (ALERT)
- net Alert: now also U4.12 (RX0)
- no-connect marks 7 -> 6
Changed lines of the file:
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@@
   (junction (at 162.56 85.09) (diameter 0) (color 0 0 0 0)
-  )
-  (junction (at 81.28 22.86) (diameter 0) (color 0 0 0 0)
   )
   (junction (at 52.07 129.54) (diameter 0) (color 0 0 0 0)
@@
   (no_connect (at 182.88 144.78))
   (no_connect (at 50.8 12.7))
-  (no_connect (at 107.95 83.82))
   (no_connect (at 25.4 165.1))
   (no_connect (at 80.01 124.46))
@@
     (stroke (width 0) (type default))
   )
-  (wire (pts (xy 82.55 22.86) (xy 81.28 22.86))
-    (stroke (width 0) (type default))
-  )
   (wire (pts (xy 133.35 78.74) (xy 133.35 81.28))
     (stroke (width 0) (type default))
@@
     (stroke (width 0) (type default))
   )
-  (wire (pts (xy 81.28 22.86) (xy 81.28 21.59))
-    (stroke (width 0) (type default))
-  )
   (wire (pts (xy 69.85 212.09) (xy 71.12 212.09))
     (stroke (width 0) (type default))
@@
   )
   (wire (pts (xy 74.93 101.6) (xy 80.01 101.6))
-    (stroke (width 0) (type default))
-  )
-  (wire (pts (xy 81.28 22.86) (xy 81.28 24.13))
     (stroke (width 0) (type default))
   )
@@
     )
   )
-  (global_label "Luminodiodes" (shape output) (at 82.55 22.86 0) (fields_autoplaced)
-    (effects (font (size 1.27 1.27)) (justify left))
-    (property "Intersheetrefs" "${INTERSHEET_REFS}" (at 98.3975 22.86 0)
+  (global_label "Alert" (shape input) (at 81.28 21.59 0) (fields_autoplaced)
+    (effects (font (size 1.27 1.27)) (justify left))
+    (property "Intersheetrefs" "${INTERSHEET_REFS}" (at 88.5401 21.59 0)
+      (effects (font (size 1.27 1.27)) (justify left) hide)
+    )
+  )
+  (global_label "Luminodiodes" (shape output) (at 81.28 24.13 0) (fields_autoplaced)
+    (effects (font (size 1.27 1.27)) (justify left))
+    (property "Intersheetrefs" "${INTERSHEET_REFS}" (at 97.1275 24.13 0)
       (effects (font (size 1.27 1.27)) (justify left) hide)
     )
@@
     )
   )
+  (global_label "Alert" (shape output) (at 107.95 83.82 180) (fields_autoplaced)
+    (effects (font (size 1.27 1.27)) (justify right))
+    (property "Intersheetrefs" "${INTERSHEET_REFS}" (at 100.6899 83.82 0)
+      (effects (font (size 1.27 1.27)) (justify right) hide)
+    )
+  )
