File: project_kicad/strange_games.kicad_pcb (KiCad board)
At the start: 2 copper layers, 330 x 247.5 mm, 150 parts, among them J1 Display, J2 Conn_02x02, J3 Conn_02x02, Q1 Si2302A, Q2 Si2302A, SW1 SW_Push, SW10 SW_Push, SW11 SW_Push, SW12 SW_Push, SW2 SW_Push, SW3 SW_Push, SW4 SW_Push, SW5 SW_Push, SW6 SW_Push, SW7 SW_Push, SW8 SW_Push, SW9 SW_Push, U1 STM32F446ZET6, U2 charge controller, U3 boost converter, U4 LDL1117S33R, U5 MQ-135 gas sensor, U6 TMP112xxDRL, U7 LSM6DS3, U8 ESP8266-01

Commit message: replaces stm32 with esp32
remade schematic, replacing stm32 with esp32, starting making pcb. Deleted projects for stm32 and esp8266
Parts:
- removed C10, C11, C12, C13, C14, C15, C16, C18, C19, C20, C42, C43, C45, C6, C68, C7, C8: C_Generic, PCM_Capacitor_SMD_AKL:C_0402_1005Metric
- removed C17, C66, C9: C_Generic, PCM_Capacitor_SMD_AKL:C_0805_2012Metric
- removed FB1: FerriteBead, Inductor_SMD:L_0805_2012Metric
- removed J2, J3: Conn_02x02, Connector_PinHeader_2.54mm:PinHeader_2x02_P2.54mm_Vertical
- removed Q1, Q2: Si2302A, Package_TO_SOT_SMD:SOT-23-3
- removed R1, R15, R19, R2, R22, R23, R24, R4, R5: 10k_0805, PCM_4ms_Resistor:R_0805_2012Metric
- removed U1: STM32F446ZET6, Package_QFP:LQFP-144_20x20mm_P0.5mm
- removed U2: charge controller, Library:charge_controller_module_tp4056
- removed U3: boost converter, Library:CKCS BS-01 MT-3608 Boost Converter
- removed U6: TMP112xxDRL, Package_TO_SOT_SMD:SOT-563
- added C70: C_Generic, PCM_Capacitor_SMD_AKL:C_0402_1005Metric, F.Cu at (187.9, 156.8)
- added C71: C_Generic, PCM_Capacitor_SMD_AKL:C_0402_1005Metric, F.Cu at (172.0, 187.0)
- added C72: C_Generic, PCM_Capacitor_SMD_AKL:C_0805_2012Metric, F.Cu at (180.8, 189.4)
- added Q3: Si2302A, Package_TO_SOT_SMD:SOT-23-3, F.Cu at (319.0, 173.0)
- added Q4: Si2302A, Package_TO_SOT_SMD:SOT-23-3, F.Cu at (319.0, 177.4)
- added R41: 10k_0805, PCM_4ms_Resistor:R_0805_2012Metric, F.Cu at (199.9, 237.2)
- added R42: 10k_0805, PCM_4ms_Resistor:R_0805_2012Metric, F.Cu at (204.3, 216.6)
- added R43: 10k_0805, PCM_4ms_Resistor:R_0805_2012Metric, F.Cu at (170.7, 175.2)
- added R44: 10k_0805, PCM_4ms_Resistor:R_0805_2012Metric, F.Cu at (170.7, 178.1)
- added R45: 10k_0805, PCM_4ms_Resistor:R_0805_2012Metric, F.Cu at (193.0, 120.2)
- added R46: 10k_0805, PCM_4ms_Resistor:R_0805_2012Metric, F.Cu at (193.0, 123.1)
- added R47: 10k_0805, PCM_4ms_Resistor:R_0805_2012Metric, F.Cu at (193.0, 126.1)
- added U9: ESP32-DEVKIT-V1, SnapEDA Library:MODULE_ESP32_DEVKIT_V1, F.Cu at (145.0, 157.5)
- C1, C3, C32, C33, C39, C4, C41, C67: footprint PCM_Capacitor_SMD_AKL:C_0402_1005Metric -> PCM_Capacitor_SMD_AKL:C_0805_2012Metric
- C21, C22, C36, C37, C64, C65: footprint PCM_Capacitor_SMD_AKL:C_0805_2012Metric -> PCM_Capacitor_SMD_AKL:C_0402_1005Metric
- D13: value S07B-GS08 -> yf923; footprint Diode_SMD:D_SMF -> LED_THT:LED_D5.0mm-4_RGB
- D4: value yf923 -> S07B-GS08; footprint LED_THT:LED_D5.0mm-4_RGB -> Diode_SMD:D_SMF
- U5: footprint Library:MQ-135 gas sensor -> Connector_PinHeader_1.27mm:PinHeader_1x04_P1.27mm_Vertical
- U7: value LSM6DS3 -> TMP112xxDRL; footprint Package_LGA:LGA-14_3x2.5mm_P0.5mm_LayoutBorder3x4y -> Package_TO_SOT_SMD:SOT-563
- U8: value ESP8266-01 -> LSM6DS3; footprint SnapEDA Library:XCVR_ESP8266-01_ESP-01 -> Package_LGA:LGA-14_3x2.5mm_P0.5mm_LayoutBorder3x4y
- moved D4 266.9 mm to (347.5, 130.0)
- moved C60 252.4 mm to (72.0, 155.8)
- moved C61 252.4 mm to (72.0, 157.9)
- moved C62 252.4 mm to (72.0, 160.0)
- moved C49 249.9 mm to (68.9, 147.3)
- moved C50 249.9 mm to (68.9, 149.4)
- moved C51 249.9 mm to (68.9, 151.5)
- moved C52 249.9 mm to (68.9, 153.6)
- moved C69 249.6 mm to (77.7, 174.0)
- moved C67 245.2 mm to (86.5, 177.5)
- moved C56 241.6 mm to (72.0, 147.3)
- moved C58 241.6 mm to (72.0, 151.5)
- moved C54 229.4 mm to (195.4, 265.5)
- moved C55 229.4 mm to (195.4, 267.6)
- moved C53 229.4 mm to (195.4, 263.4)
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Connections:
- C1 pad 2: Net-(U1-VCAP_1) -> +3V3
- C2 pad 1: GND -> +3V3
- C2 pad 2: Net-(U1-VCAP_2) -> GND
- C21 pad 1: GND -> Net-(J1-CAP5+)
- C21 pad 2: VDC -> Net-(J1-CAP1-)
- C22 pad 1: GND -> Net-(J1-CAP2+)
- C22 pad 2: VDC -> Net-(J1-CAP2-)
- C23 pad 1: Net-(J1-CAP5+) -> Net-(J1-CAP4+)
- C23 pad 2: Net-(J1-CAP1-) -> Net-(J1-CAP2-)
- C24 pad 1: Net-(J1-CAP2+) -> +3V3
- C24 pad 2: Net-(J1-CAP2-) -> Net-(J1-V3)
- C25 pad 1: Net-(J1-CAP4+) -> +3V3
- C25 pad 2: Net-(J1-CAP2-) -> Net-(J1-V1)
- C26 pad 1: +3V3 -> Net-(J1-Vout)
- C26 pad 2: Net-(J1-V3) -> GND
- C27 pad 1: +3V3 -> Net-(J1-CAP3+)
- C27 pad 2: Net-(J1-V1) -> Net-(J1-CAP1-)
- C28 pad 1: Net-(J1-Vout) -> Net-(J1-CAP1+)
- C28 pad 2: GND -> Net-(J1-CAP1-)
- C29 pad 1: Net-(J1-CAP3+) -> +3V3
- C29 pad 2: Net-(J1-CAP1-) -> Net-(J1-V4)
- C30 pad 1: Net-(J1-CAP1+) -> +3V3
- C30 pad 2: Net-(J1-CAP1-) -> Net-(J1-V2)
- C31 pad 2: Net-(J1-V4) -> Net-(J1-V0)
- C32 pad 1: +3V3 -> GND
- C32 pad 2: Net-(J1-V2) -> VDC
- C33 pad 1: +3V3 -> GND
- C33 pad 2: Net-(J1-V0) -> VDC
- C35 pad 1: GND -> B10
- C36 pad 1: GND -> B11
- C36 pad 2: +12V -> +3V3
- C37 pad 1: GND -> B12
- C38 pad 1: -BATT -> GND
- C38 pad 2: +BATT -> +12V
- C39 pad 1: B10 -> GND
- C4 pad 1: +3V3 -> GND
- C4 pad 2: GND -> +3V3
- C40 pad 1: B11 -> GND
- C41 pad 1: B12 -> -BATT
- C41 pad 2: +3V3 -> +BATT
- C44 pad 1: B2 -> GND
- C46 pad 1: GND -> B1
- C47 pad 1: +3V3 -> B2
- C47 pad 2: GND -> +3V3
- C48 pad 1: GND -> B3
- C49 pad 1: +3V3 -> GND
- C49 pad 2: GND -> +3V3
- C5 pad 1: +3.3VA -> +3V3
- C50 pad 1: GND -> +3V3
- C50 pad 2: +3V3 -> GND
- C52 pad 1: GND -> +3V3
- C52 pad 2: +3V3 -> GND
- C56 pad 1: +3V3 -> GND
- C56 pad 2: GND -> +3V3
- C58 pad 1: GND -> +3V3
- C58 pad 2: +3V3 -> GND
- C59 pad 1: +3V3 -> GND
- C59 pad 2: GND -> +3V3
- C61 pad 1: B7 -> +3V3
- C61 pad 2: +3V3 -> GND
- C62 pad 1: B8 -> GND
- C63 pad 1: B9 -> B7
- C64 pad 1: GND -> B8
- C65 pad 1: GND -> B9
- C67 pad 1: +3V3 -> GND
- C67 pad 2: GND -> +3V3
- D12 pad 1: unconnected-(D12-DO-Pad1) -> Net-(D12-DO)
- D13 pad 1: VDC -> unconnected-(D13-DO-Pad1)
- D13 pad 2: +3V3 -> GND
- D2 pad 1: +12V -> VDC
- D2 pad 2: Net-(D2-A) -> +3V3
- D3 pad 1: +3V3 -> +12V
- D4 pad 1: Net-(D4-DO) -> +3V3
- D4 pad 2: GND -> Net-(D4-A)
- D5 pad 4: Net-(D10-DO) -> luminodiodes
- D7 pad 1: Net-(D10-DI) -> Net-(D12-DI)
- D7 pad 4: Net-(D4-DO) -> Net-(D6-DO)
- D9 pad 1: Net-(D12-DI) -> Net-(D10-DI)
- D9 pad 4: Net-(D6-DO) -> Net-(D12-DO)
- J1 pad 22: D10 -> SDA
- J1 pad 23: D9 -> SCL
- J1 pad 24: D8 -> unconnected-(J1-D5-Pad24)
- J1 pad 25: D7 -> unconnected-(J1-D4-Pad25)
- J1 pad 26: D6 -> unconnected-(J1-D3-Pad26)
- J1 pad 27: D5 -> unconnected-(J1-D2-Pad27)
- J1 pad 28: D4 -> unconnected-(J1-D1-Pad28)
- J1 pad 29: D3 -> unconnected-(J1-D0-Pad29)
- J1 pad 3: +3V3 -> GND
- J1 pad 30: D2 -> RD_display
- J1 pad 31: D1 -> WR_display
- J1 pad 32: D0 -> A0_display
- R10 pad 1: alert_tmp -> GND
- R10 pad 2: +3V3 -> Net-(R10-Pad2)
- R11 pad 1: NRST -> GND
- R11 pad 2: +3V3 -> Net-(R11-Pad2)
- R12 pad 1: BOOT0 -> GND
- R12 pad 2: GND -> Net-(R12-Pad2)
- R13 pad 2: С1 -> vibrating_signal
- R14 pad 1: SDA_lsm -> GND
- R14 pad 2: +3V3 -> photo_2
- R16 pad 1: SCL_lsm -> Net-(Q3-G)
- R16 pad 2: +3V3 -> open_box
- R17 pad 1: A10 -> alert_tmp
- R18 pad 1: B1 -> GND
- R18 pad 2: Net-(R18-Pad2) -> Net-(Q3-G)
- R20 pad 1: B3 -> Net-(Q4-G)
- R20 pad 2: Net-(R20-Pad2) -> vibrating_motor
- R21 pad 2: Net-(R18-Pad2) -> Net-(Q4-G)
- R25 pad 1: B5 -> B1
- R26 pad 1: B6 -> B2
- R27 pad 1: Net-(J3-+12V-Pad2) -> B3
- R27 pad 2: +3V3 -> Net-(R27-Pad2)
- R28 pad 1: unconnected-(R28-Pad1) -> GND
- R28 pad 2: Net-(R24-Pad2) -> Net-(R25-Pad2)
- R29 pad 2: Net-(R25-Pad2) -> Net-(R26-Pad2)
- R3 pad 1: B11 -> GND
- R3 pad 2: Net-(R3-Pad2) -> gas_signal
- R30 pad 2: Net-(R26-Pad2) -> Net-(R27-Pad2)
- R31 pad 1: B7 -> B4
- R32 pad 1: B8 -> B5
- R33 pad 1: B9 -> B6
- R34 pad 1: unconnected-(R34-Pad1) -> GND
- R37 pad 1: CS_lsm -> B7
- R37 pad 2: +3V3 -> Net-(R37-Pad2)
- R38 pad 1: GND -> B8
- R38 pad 2: C2 -> Net-(R38-Pad2)
- R39 pad 1: GND -> B9
- R39 pad 2: С3 -> Net-(R39-Pad2)
- R40 pad 1: GND -> unconnected-(R40-Pad1)
- R40 pad 2: С4 -> Net-(R37-Pad2)
- R6 pad 1: GND -> B10
- R6 pad 2: Net-(R2-Pad2) -> Net-(R10-Pad2)
- R7 pad 1: GND -> B11
- R7 pad 2: Net-(R3-Pad2) -> Net-(R11-Pad2)
- R8 pad 1: GND -> B12
- R8 pad 2: Net-(R4-Pad2) -> Net-(R12-Pad2)
- R9 pad 1: SCL_tmp -> GND
- R9 pad 2: +3V3 -> photo_1
- SW1 pad 2: Net-(R2-Pad2) -> Net-(R10-Pad2)
- SW10 pad 2: Net-(R31-Pad2) -> Net-(R37-Pad2)
- SW11 pad 2: Net-(R32-Pad2) -> Net-(R38-Pad2)
- SW12 pad 2: Net-(R33-Pad2) -> Net-(R39-Pad2)
- SW2 pad 2: Net-(R3-Pad2) -> Net-(R11-Pad2)
- SW3 pad 2: Net-(R4-Pad2) -> Net-(R12-Pad2)
- SW4 pad 2: Net-(R18-Pad2) -> Net-(R25-Pad2)
- SW5 pad 2: Net-(R19-Pad2) -> Net-(R26-Pad2)
- SW6 pad 2: Net-(R20-Pad2) -> Net-(R27-Pad2)
- SW7 pad 2: Net-(R24-Pad2) -> Net-(R31-Pad2)
- SW8 pad 2: Net-(R25-Pad2) -> Net-(R32-Pad2)
- SW9 pad 2: Net-(R26-Pad2) -> Net-(R33-Pad2)
- U5 pad 1: GND -> +3V3
- U5 pad 2: +3V3 -> GND
- U5 pad 3: C15 -> gas_signal
- U5 pad 4: (no net) -> unconnected-(U5-AO-Pad4)
- U7 pad 1: GND -> SCL
- U7 pad 2: unconnected-(U7-SDX-Pad2) -> GND
- U7 pad 3: unconnected-(U7-SCX-Pad3) -> alert_tmp
- U7 pad 4: INT1_LSM -> GND
- U7 pad 6: GND -> SDA
- U8 pad 2: Net-(U8-IO2) -> unconnected-(U8-SDX-Pad2)
- U8 pad 3: Net-(U8-IO0) -> unconnected-(U8-SCX-Pad3)
- U8 pad 4: A9 -> INT1_LSM
- U8 pad 5: A10 -> +3V3
- U8 pad 6: Net-(U8-EN) -> GND
- U8 pad 7: Net-(U8-~{RST}) -> GND
Routing:
- removed copper zone on B.Cu, net GND

Commit message: some more changes in sch
Parts:
- removed C22, C24, C25, C54, C55, C56, C57, C58, C59, C60, C61, C62, C63, C64, C65, C69, C70, C71: C_Generic, PCM_Capacitor_SMD_AKL:C_0402_1005Metric
- removed C67, C72: C_Generic, PCM_Capacitor_SMD_AKL:C_0805_2012Metric
- removed R10, R11, R17, R39, R40, R41, R42, R43, R44, R45, R46, R47, R7, R8: 10k_0805, PCM_4ms_Resistor:R_0805_2012Metric
- removed SW2, SW3: SW_Push, Button_Switch_THT:SW_PUSH-12mm
- removed U9: ESP32-DEVKIT-V1, SnapEDA Library:MODULE_ESP32_DEVKIT_V1
- added C10: C_Generic, PCM_Capacitor_SMD_AKL:C_0402_1005Metric, F.Cu at (213.3, 161.9)
- added C11: C_Generic, PCM_Capacitor_SMD_AKL:C_0402_1005Metric, F.Cu at (213.3, 164.1)
- added C12: C_Generic, PCM_Capacitor_SMD_AKL:C_0402_1005Metric, F.Cu at (213.3, 166.2)
- added C13: C_Generic, PCM_Capacitor_SMD_AKL:C_0402_1005Metric, F.Cu at (216.4, 155.6)
- added C14: C_Generic, PCM_Capacitor_SMD_AKL:C_0402_1005Metric, F.Cu at (216.4, 157.7)
- added C15: C_Generic, PCM_Capacitor_SMD_AKL:C_0402_1005Metric, F.Cu at (216.4, 159.8)
- added C16: C_Generic, PCM_Capacitor_SMD_AKL:C_0402_1005Metric, F.Cu at (216.4, 161.9)
- added C17: C_Generic, PCM_Capacitor_SMD_AKL:C_0402_1005Metric, F.Cu at (216.4, 164.1)
- added C18: C_Generic, PCM_Capacitor_SMD_AKL:C_0402_1005Metric, F.Cu at (216.4, 166.2)
- added C19: C_Generic, PCM_Capacitor_SMD_AKL:C_0805_2012Metric, F.Cu at (275.9, 183.0)
- added C20: C_Generic, PCM_Capacitor_SMD_AKL:C_0805_2012Metric, F.Cu at (214.2, 175.0)
- added C42: C_Generic, PCM_Capacitor_SMD_AKL:C_0402_1005Metric, F.Cu at (219.6, 155.6)
- added C43: C_Generic, PCM_Capacitor_SMD_AKL:C_0402_1005Metric, F.Cu at (219.6, 157.7)
- added C45: C_Generic, PCM_Capacitor_SMD_AKL:C_0402_1005Metric, F.Cu at (219.6, 159.8)
- added C6: C_Generic, PCM_Capacitor_SMD_AKL:C_0805_2012Metric, F.Cu at (214.2, 168.8)
- added C7: C_Generic, PCM_Capacitor_SMD_AKL:C_0402_1005Metric, F.Cu at (213.3, 155.6)
- added C8: C_Generic, PCM_Capacitor_SMD_AKL:C_0402_1005Metric, F.Cu at (213.3, 157.7)
- added C9: C_Generic, PCM_Capacitor_SMD_AKL:C_0402_1005Metric, F.Cu at (213.3, 159.8)
- added Q1: Si2302A, Package_TO_SOT_SMD:SOT-23-3, F.Cu at (223.7, 173.6)
- added R1: 10k_0805, PCM_4ms_Resistor:R_0805_2012Metric, F.Cu at (223.3, 156.0)
- added R15: 10k_0805, PCM_4ms_Resistor:R_0805_2012Metric, F.Cu at (227.7, 158.9)
- added R19: 10k_0805, PCM_4ms_Resistor:R_0805_2012Metric, F.Cu at (227.7, 161.9)
- added R2: 10k_0805, PCM_4ms_Resistor:R_0805_2012Metric, F.Cu at (223.3, 158.9)
- added R22: 10k_0805, PCM_4ms_Resistor:R_0805_2012Metric, F.Cu at (232.1, 156.0)
- added R23: 10k_0805, PCM_4ms_Resistor:R_0805_2012Metric, F.Cu at (232.1, 158.9)
- added R24: 10k_0805, PCM_4ms_Resistor:R_0805_2012Metric, F.Cu at (232.1, 161.9)
- added R4: 10k_0805, PCM_4ms_Resistor:R_0805_2012Metric, F.Cu at (223.3, 161.9)
- added R5: 10k_0805, PCM_4ms_Resistor:R_0805_2012Metric, F.Cu at (227.7, 156.0)
- added U3: LDL1117S33R, SnapEDA Library:SOT230P700X180-4N, F.Cu at (277.2, 175.6)
- C2, C21, C37, C49: footprint PCM_Capacitor_SMD_AKL:C_0402_1005Metric -> PCM_Capacitor_SMD_AKL:C_0805_2012Metric
- C32, C33, C34, C38, C39, C41: footprint PCM_Capacitor_SMD_AKL:C_0805_2012Metric -> PCM_Capacitor_SMD_AKL:C_0402_1005Metric
- U4: value LDL1117S33R -> ESP32-DEVKIT-V1; footprint SnapEDA Library:SOT230P700X180-4N -> SnapEDA Library:MODULE_ESP32_DEVKIT_V1
- U5: value MQ-135 gas sensor -> TMP112xxDRL; footprint Connector_PinHeader_1.27mm:PinHeader_1x04_P1.27mm_Vertical -> Package_TO_SOT_SMD:SOT-563
- U7: value TMP112xxDRL -> LSM6DS3; footprint Package_TO_SOT_SMD:SOT-563 -> Package_LGA:LGA-14_3x2.5mm_P0.5mm_LayoutBorder3x4y
- U8: value LSM6DS3 -> MQ-135 gas sensor; footprint Package_LGA:LGA-14_3x2.5mm_P0.5mm_LayoutBorder3x4y -> Connector_PinHeader_1.27mm:PinHeader_1x04_P1.27mm_Vertical
- moved C21 119.5 mm to (275.9, 185.3)
- moved U4 93.9 mm to (150.4, 159.5)
- moved C4 92.8 mm to (270.8, 180.7)
- moved D2 36.5 mm to (275.4, 180.7)
Connections:
- net VR renamed Net-(J1-VR)
- C2 pad 1: +3V3 -> GND
- C2 pad 2: GND -> +3V3
- C21 pad 1: Net-(J1-CAP5+) -> GND
- C21 pad 2: Net-(J1-CAP1-) -> +3V3
- C23 pad 1: Net-(J1-CAP4+) -> B10
- C23 pad 2: Net-(J1-CAP2-) -> +3V3
- C26 pad 1: Net-(J1-Vout) -> B1
- C26 pad 2: GND -> +3V3
- C27 pad 1: Net-(J1-CAP3+) -> B2
- C27 pad 2: Net-(J1-CAP1-) -> +3V3
- C28 pad 1: Net-(J1-CAP1+) -> B3
- C28 pad 2: Net-(J1-CAP1-) -> +3V3
- C29 pad 1: +3V3 -> B4
- C29 pad 2: Net-(J1-V4) -> +3V3
- C3 pad 2: +3V3 -> VDC
- C30 pad 1: +3V3 -> B5
- C30 pad 2: Net-(J1-V2) -> +3V3
- C31 pad 1: +3V3 -> B6
- C31 pad 2: Net-(J1-V0) -> +3V3
- C32 pad 2: VDC -> +3V3
- C33 pad 1: GND -> +3V3
- C33 pad 2: VDC -> GND
- C35 pad 1: B10 -> +3V3
- C35 pad 2: +3V3 -> GND
- C36 pad 1: B11 -> GND
- C37 pad 1: B12 -> GND
- C38 pad 2: +12V -> +3V3
- C39 pad 1: GND -> B7
- C4 pad 2: +3V3 -> VDC
- C40 pad 1: GND -> B8
- C41 pad 1: -BATT -> B9
- C41 pad 2: +BATT -> +3V3
- C46 pad 1: B1 -> GND
- C47 pad 1: B2 -> GND
- C48 pad 1: B3 -> GND
- C51 pad 1: GND -> +3V3
- C51 pad 2: +3V3 -> GND
- C52 pad 1: +3V3 -> GND
- C52 pad 2: GND -> +3V3
- C53 pad 1: B4 -> GND
- D7 pad 1: Net-(D12-DI) -> Net-(D10-DI)
- D7 pad 4: Net-(D6-DO) -> Net-(D12-DO)
- D9 pad 1: Net-(D10-DI) -> Net-(D12-DI)
- D9 pad 4: Net-(D12-DO) -> Net-(D6-DO)
- Q3 pad 3: Net-(D3-A) -> Net-(D4-A)
- R12 pad 1: GND -> Net-(Q1-G)
- R12 pad 2: Net-(R12-Pad2) -> open_box
- R13 pad 2: vibrating_signal -> Net-(Q1-G)
- R14 pad 1: GND -> Net-(Q3-G)
- R14 pad 2: photo_2 -> vibrating_motor
- R16 pad 1: Net-(Q3-G) -> GND
- R16 pad 2: open_box -> photo_1
- R18 pad 1: GND -> B1
- R18 pad 2: Net-(Q3-G) -> Net-(R18-Pad2)
- R20 pad 1: Net-(Q4-G) -> B3
- R20 pad 2: vibrating_motor -> Net-(R20-Pad2)
- R21 pad 2: Net-(Q4-G) -> photo_2
- R25 pad 1: B1 -> GND
- R25 pad 2: Net-(R25-Pad2) -> vibrating_signal
- R26 pad 1: B2 -> B4
- R27 pad 1: B3 -> B5
- R28 pad 1: GND -> B6
- R28 pad 2: Net-(R25-Pad2) -> Net-(R28-Pad2)
- R3 pad 1: GND -> A0_display
- R3 pad 2: gas_signal -> +3V3
- R31 pad 1: B4 -> GND
- R31 pad 2: Net-(R31-Pad2) -> Net-(R28-Pad2)
- R32 pad 1: B5 -> GND
- R32 pad 2: Net-(R32-Pad2) -> gas_signal
- R33 pad 1: B6 -> B7
- R34 pad 1: GND -> B8
- R34 pad 2: Net-(R31-Pad2) -> Net-(R34-Pad2)
- R35 pad 1: GND -> B9
- R35 pad 2: Net-(R32-Pad2) -> Net-(R35-Pad2)
- R36 pad 1: GND -> unconnected-(R36-Pad1)
- R37 pad 1: B7 -> GND
- R37 pad 2: Net-(R37-Pad2) -> Net-(R34-Pad2)
- R38 pad 1: B8 -> GND
- R38 pad 2: Net-(R38-Pad2) -> Net-(R35-Pad2)
- R6 pad 2: Net-(R10-Pad2) -> Net-(R6-Pad2)
- R9 pad 2: photo_1 -> Net-(R6-Pad2)
- SW1 pad 2: Net-(R10-Pad2) -> Net-(R6-Pad2)
- SW10 pad 2: Net-(R37-Pad2) -> Net-(R33-Pad2)
- SW11 pad 2: Net-(R38-Pad2) -> Net-(R34-Pad2)
- SW12 pad 2: Net-(R39-Pad2) -> Net-(R35-Pad2)
- SW4 pad 2: Net-(R25-Pad2) -> Net-(R18-Pad2)
- SW5 pad 2: Net-(R26-Pad2) -> Net-(R19-Pad2)
- SW6 pad 2: Net-(R27-Pad2) -> Net-(R20-Pad2)
- SW7 pad 2: Net-(R31-Pad2) -> Net-(R26-Pad2)
- SW8 pad 2: Net-(R32-Pad2) -> Net-(R27-Pad2)
- SW9 pad 2: Net-(R33-Pad2) -> Net-(R28-Pad2)
- U4 pad 1: GND -> +3V3
- U4 pad 2: +3V3 -> GND
- U4 pad 3: VDC -> A0_display
- U4 pad 4: +3V3 -> luminodiodes
- U5 pad 1: +3V3 -> SCL
- U5 pad 3: gas_signal -> unconnected-(U5-ALERT-Pad3)
- U5 pad 4: unconnected-(U5-AO-Pad4) -> GND
- U7 pad 1: SCL -> GND
- U7 pad 2: GND -> unconnected-(U7-SDX-Pad2)
- U7 pad 3: alert_tmp -> unconnected-(U7-SCX-Pad3)
- U7 pad 4: GND -> INT1
- U7 pad 6: SDA -> GND
- U8 pad 1: GND -> +3V3
- U8 pad 2: unconnected-(U8-SDX-Pad2) -> GND
- U8 pad 3: unconnected-(U8-SCX-Pad3) -> gas_signal
- U8 pad 4: INT1_LSM -> unconnected-(U8-AO-Pad4)
Routing:
- net +3V3: track 0.00 -> 17.0 mm
- net VDC: track 0.00 -> 4.99 mm

Commit message: updated placements for pcb
Parts:
- added L1: L_Iron, Connector_PinHeader_2.54mm:PinHeader_1x02_P2.54mm_Vertical, F.Cu at (335.8, 183.9)
- added M1: Motor_DC, Connector_PinHeader_2.54mm:PinHeader_1x02_P2.54mm_Vertical, F.Cu at (335.8, 174.8)
- added Q2: Q_Photo, LED_THT:LED_D4.0mm, F.Cu at (326.4, 177.8)
- added U1: charge controller, SnapEDA Library:charge_controller_module_tp4056, F.Cu at (237.1, 187.2)
- added U2: boost converter, SnapEDA Library:CKCS BS-01 MT-3608 Boost Converter, F.Cu at (255.4, 182.4)
- added U6: vibrating_sensor, Connector_PinHeader_2.54mm:PinHeader_1x03_P2.54mm_Vertical, F.Cu at (343.9, 181.6)
- Q4: value Si2302A -> Q_Photo; footprint Package_TO_SOT_SMD:SOT-23-3 -> LED_THT:LED_D4.0mm
- moved C39 27.5 mm to (287.4, 153.4)
- moved C41 27.5 mm to (287.4, 156.5)
- moved C38 27.5 mm to (277.0, 166.1)
- moved C33 27.5 mm to (282.5, 162.7)
- moved C34 27.5 mm to (282.5, 165.9)
- moved C32 27.5 mm to (282.5, 159.6)
- moved Q4 10.3 mm to (326.1, 184.9)
- moved C10 4.93 mm to (213.3, 157.0)
- moved C14 4.93 mm to (216.4, 152.8)
- moved C15 4.93 mm to (216.4, 154.9)
- moved C16 4.93 mm to (216.4, 157.0)
- moved C20 4.93 mm to (214.2, 170.1)
- moved C43 4.93 mm to (219.6, 152.8)
- moved C45 4.93 mm to (219.6, 154.9)
- moved C8 4.93 mm to (213.3, 152.8)
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Connections:
- Q4 pad 1: Net-(Q4-G) -> +3V3
- Q4 pad 2: GND -> photo_2

Commit message: pcb changes
Parts:
- D10, D11, D12, D13, D5, D6, D7, D8, D9, Q2, Q4, SW1, SW10, SW11, SW12, SW4, SW5, SW6, SW7, SW8, SW9: moved to B.Cu
- moved SW10 52.4 mm to (187.8, 221.6), turned to 180 degrees
- moved SW11 52.4 mm to (187.8, 235.1), turned to 180 degrees
- moved SW12 52.4 mm to (187.8, 248.7), turned to 180 degrees
- moved D6 42.6 mm to (105.1, 127.5), turned to 180 degrees
- moved D7 42.6 mm to (105.1, 135.1), turned to 180 degrees
- moved D5 35.0 mm to (66.3, 127.9), turned to 180 degrees
- moved D8 27.5 mm to (97.5, 127.5), turned to 180 degrees
- moved D9 27.5 mm to (97.5, 135.1), turned to 180 degrees
- moved SW7 24.4 mm to (149.4, 216.2), turned to 180 degrees
- moved SW8 24.4 mm to (149.4, 233.7), turned to 180 degrees
- moved SW9 24.4 mm to (149.4, 251.2), turned to 180 degrees
- moved SW4 15.6 mm to (169.4, 216.2), turned to 180 degrees
- moved SW5 15.6 mm to (169.4, 233.7), turned to 180 degrees
- moved SW6 15.6 mm to (169.4, 251.2), turned to 180 degrees
- moved D10 12.4 mm to (90.0, 127.5), turned to 180 degrees
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
Commit message: updated buttons
Parts:
- moved C23 319.3 mm to (459.6, 269.1)
- moved C36 319.3 mm to (465.9, 260.7)
- moved C46 316.0 mm to (502.5, 323.3)
- moved C48 316.0 mm to (502.5, 327.5)
- moved C53 316.0 mm to (505.6, 323.3)
- moved R32 316.0 mm to (505.7, 294.2)
- moved R25 315.3 mm to (501.3, 293.5)
- moved R18 285.7 mm to (76.0, 264.0), turned to 180 degrees
- moved R22 194.2 mm to (76.0, 266.5), turned to 180 degrees
- moved R20 180.3 mm to (166.6, 212.5)
- moved C32 174.3 mm to (108.4, 150.0)
- moved C33 174.3 mm to (108.4, 153.1)
- moved C34 174.3 mm to (108.4, 156.2)
- moved C26 171.1 mm to (79.0, 263.9)
- moved C47 142.4 mm to (85.9, 170.9)
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Routing:
- net Net-(R18-Pad2): track 0.00 -> 12.6 mm
- net +3V3: track 17.0 -> 29.5 mm
- net B1: track 0.00 -> 1.48 mm

Commit message: updated pcb
Parts:
- removed C10, C36, C44, C5, C51, C52, C53, C8: C_Generic, PCM_Capacitor_SMD_AKL:C_0402_1005Metric
- removed R34, R35, R36, R37, R38: 10k_0805, PCM_4ms_Resistor:R_0805_2012Metric
- removed SW11, SW12: SW_Push, Button_Switch_THT:SW_PUSH-12mm
- added C22: C_Generic, PCM_Capacitor_SMD_AKL:C_0402_1005Metric, F.Cu at (264.2, 208.9)
- added C24: C_Generic, PCM_Capacitor_SMD_AKL:C_0402_1005Metric, F.Cu at (148.3, 210.0)
- added C25: C_Generic, PCM_Capacitor_SMD_AKL:C_0402_1005Metric, F.Cu at (168.3, 210.0)
- added R10: 10k_0805, PCM_4ms_Resistor:R_0805_2012Metric, F.Cu at (260.4, 215.2)
- added R11: 10k_0805, PCM_4ms_Resistor:R_0805_2012Metric, F.Cu at (260.4, 218.2)
- added R17: 10k_0805, PCM_4ms_Resistor:R_0805_2012Metric, F.Cu at (151.1, 212.5)
- added R7: 10k_0805, PCM_4ms_Resistor:R_0805_2012Metric, F.Cu at (260.4, 209.3)
- added R8: 10k_0805, PCM_4ms_Resistor:R_0805_2012Metric, F.Cu at (260.4, 212.3)
- added SW2: SW_Push, Button_Switch_THT:SW_PUSH-12mm, B.Cu at (147.5, 207.1)
- added SW3: SW_Push, Button_Switch_THT:SW_PUSH-12mm, B.Cu at (167.5, 207.1)
- C1, C19, C20, C21, C37, C49, C6: footprint PCM_Capacitor_SMD_AKL:C_0805_2012Metric -> PCM_Capacitor_SMD_AKL:C_0402_1005Metric
- C11, C12, C33, C41, C7: footprint PCM_Capacitor_SMD_AKL:C_0402_1005Metric -> PCM_Capacitor_SMD_AKL:C_0805_2012Metric
- moved C46 461.0 mm to (65.8, 175.6), turned to 90 degrees
- moved R32 337.2 mm to (171.1, 252.5)
- moved R25 335.8 mm to (171.1, 232.5)
- moved C48 259.9 mm to (264.2, 223.8)
- moved C23 203.9 mm to (264.2, 211.1)
- moved R21 200.7 mm to (151.1, 230.0)
- moved R14 182.6 mm to (171.1, 210.0)
- moved C38 137.3 mm to (168.3, 250.0), turned to 180 degrees
- moved SW4 126.6 mm to (187.5, 207.1), turned to -90 degrees
- moved C26 121.9 mm to (188.3, 210.0), turned to 180 degrees
- moved C30 118.9 mm to (65.8, 135.6), turned to 90 degrees
- moved R18 108.1 mm to (171.1, 212.5), turned to 0 degrees
- moved C31 106.3 mm to (85.8, 135.6), turned to -90 degrees
- moved C37 106.3 mm to (148.3, 250.0), turned to 180 degrees
- moved R22 101.9 mm to (171.1, 230.0), turned to 0 degrees
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Connections:
- C11 pad 1: +3V3 -> GND
- C11 pad 2: Net-(J1-V3) -> +12V
- C12 pad 1: +3V3 -> GND
- C12 pad 2: Net-(J1-V1) -> +3V3
- C13 pad 1: Net-(J1-Vout) -> Net-(J1-CAP5+)
- C13 pad 2: GND -> Net-(J1-CAP1-)
- C14 pad 1: Net-(J1-CAP3+) -> Net-(J1-CAP2+)
- C14 pad 2: Net-(J1-CAP1-) -> Net-(J1-CAP2-)
- C15 pad 1: Net-(J1-CAP1+) -> Net-(J1-CAP4+)
- C15 pad 2: Net-(J1-CAP1-) -> Net-(J1-CAP2-)
- C16 pad 2: Net-(J1-V4) -> Net-(J1-V3)
- C17 pad 2: Net-(J1-V2) -> Net-(J1-V1)
- C18 pad 1: +3V3 -> Net-(J1-Vout)
- C18 pad 2: Net-(J1-V0) -> GND
- C19 pad 1: GND -> Net-(J1-CAP3+)
- C19 pad 2: +3V3 -> Net-(J1-CAP1-)
- C20 pad 1: GND -> Net-(J1-CAP1+)
- C20 pad 2: +12V -> Net-(J1-CAP1-)
- C21 pad 1: GND -> +3V3
- C21 pad 2: +3V3 -> Net-(J1-V4)
- C23 pad 1: B10 -> +3V3
- C23 pad 2: +3V3 -> Net-(J1-V0)
- C26 pad 1: B1 -> B3
- C27 pad 1: B2 -> B4
- C28 pad 1: B3 -> B5
- C29 pad 1: B4 -> B6
- C30 pad 1: B5 -> GND
- C31 pad 1: B6 -> +3V3
- C31 pad 2: +3V3 -> GND
- C33 pad 1: +3V3 -> GND
- C33 pad 2: GND -> +3V3
- C34 pad 1: GND -> +3V3
- C34 pad 2: +3V3 -> GND
- C35 pad 1: +3V3 -> GND
- C35 pad 2: GND -> +3V3
- C37 pad 1: GND -> B7
- C38 pad 1: GND -> B8
- C39 pad 1: B7 -> B9
- C40 pad 1: B8 -> GND
- C41 pad 1: B9 -> GND
- C45 pad 1: +3V3 -> GND
- C45 pad 2: GND -> +3V3
- C49 pad 1: GND -> +3V3
- C49 pad 2: +3V3 -> GND
- C50 pad 1: +3V3 -> GND
- C50 pad 2: GND -> +3V3
- C6 pad 1: GND -> B10
- C7 pad 1: +3V3 -> GND
- C7 pad 2: GND -> +3V3
- C9 pad 1: Net-(J1-CAP2+) -> GND
- C9 pad 2: Net-(J1-CAP2-) -> +3V3
- D11 pad 4: Net-(D11-DI) -> Net-(D10-DO)
- D12 pad 4: Net-(D12-DI) -> Net-(D11-DO)
- D13 pad 4: Net-(D10-DO) -> Net-(D12-DO)
- D6 pad 4: Net-(D11-DO) -> Net-(D5-DO)
- D7 pad 1: Net-(D10-DI) -> Net-(D7-DO)
- D7 pad 4: Net-(D12-DO) -> Net-(D6-DO)
- D8 pad 1: Net-(D11-DI) -> Net-(D8-DO)
- D8 pad 4: Net-(D5-DO) -> Net-(D7-DO)
- D9 pad 1: Net-(D12-DI) -> Net-(D10-DI)
- D9 pad 4: Net-(D6-DO) -> Net-(D8-DO)
- R12 pad 1: Net-(Q1-G) -> GND
- R12 pad 2: open_box -> photo_1
- R13 pad 1: GND -> B1
- R13 pad 2: Net-(Q1-G) -> Net-(R13-Pad2)
- R14 pad 1: Net-(Q3-G) -> B2
- R14 pad 2: vibrating_motor -> Net-(R14-Pad2)
- R15 pad 1: GND -> B3
- R15 pad 2: Net-(Q3-G) -> Net-(R15-Pad2)
- R16 pad 2: photo_1 -> photo_2
- R18 pad 1: B1 -> GND
- R18 pad 2: Net-(R18-Pad2) -> Net-(R14-Pad2)
- R19 pad 1: B2 -> GND
- R19 pad 2: Net-(R19-Pad2) -> Net-(R15-Pad2)
- R20 pad 1: B3 -> GND
- R20 pad 2: Net-(R20-Pad2) -> vibrating_signal
- R21 pad 1: GND -> B4
- R21 pad 2: photo_2 -> Net-(R21-Pad2)
- R22 pad 1: GND -> B5
- R22 pad 2: Net-(R18-Pad2) -> Net-(R22-Pad2)
- R23 pad 1: GND -> B6
- R23 pad 2: Net-(R19-Pad2) -> Net-(R23-Pad2)
- R24 pad 2: Net-(R20-Pad2) -> Net-(R21-Pad2)
- R25 pad 2: vibrating_signal -> Net-(R22-Pad2)
- R26 pad 1: B4 -> GND
- R26 pad 2: Net-(R26-Pad2) -> Net-(R23-Pad2)
- R27 pad 1: B5 -> GND
- R27 pad 2: Net-(R27-Pad2) -> gas_signal
- R28 pad 1: B6 -> B7
- R29 pad 1: GND -> B8
- R29 pad 2: Net-(R26-Pad2) -> Net-(R29-Pad2)
- R3 pad 1: A0_display -> B10
- R3 pad 2: +3V3 -> Net-(R3-Pad2)
- R30 pad 1: GND -> B9
- R30 pad 2: Net-(R27-Pad2) -> Net-(R30-Pad2)
- R31 pad 1: GND -> unconnected-(R31-Pad1)
- R32 pad 2: gas_signal -> Net-(R29-Pad2)
- R33 pad 1: B7 -> GND
- R33 pad 2: Net-(R33-Pad2) -> Net-(R30-Pad2)
- R4 pad 1: WR_display -> GND
- R4 pad 2: +3V3 -> Net-(R3-Pad2)
- R5 pad 1: RD_display -> A0_display
- R6 pad 1: B10 -> WR_display
- R6 pad 2: Net-(R6-Pad2) -> +3V3
- R9 pad 2: Net-(R6-Pad2) -> Net-(Q1-G)
- SW1 pad 2: Net-(R6-Pad2) -> Net-(R3-Pad2)
- SW10 pad 2: Net-(R33-Pad2) -> Net-(R30-Pad2)
- SW4 pad 2: Net-(R18-Pad2) -> Net-(R15-Pad2)
- SW5 pad 2: Net-(R19-Pad2) -> Net-(R21-Pad2)
- SW6 pad 2: Net-(R20-Pad2) -> Net-(R22-Pad2)
- SW7 pad 2: Net-(R26-Pad2) -> Net-(R23-Pad2)
- SW8 pad 2: Net-(R27-Pad2) -> Net-(R28-Pad2)
- SW9 pad 2: Net-(R28-Pad2) -> Net-(R29-Pad2)
Routing:
- net +3V3: track 29.5 -> 289.2 mm
- net Net-(D7-DO): track 0.00 -> 54.4 mm
- net Net-(D10-DO): track 0.00 -> 53.2 mm
- net Net-(D8-DO): track 0.00 -> 16.2 mm
- net Net-(D6-DO): track 0.00 -> 16.2 mm
- net Net-(D5-DO): track 0.00 -> 16.2 mm
- net Net-(D12-DO): track 0.00 -> 16.2 mm
- net Net-(D11-DO): track 0.00 -> 16.2 mm
- net Net-(D10-DI): track 0.00 -> 16.2 mm
- net Net-(R18-Pad2): track 12.6 -> 0.00 mm
- net Net-(R30-Pad2): track 0.00 -> 12.5 mm
- net Net-(R3-Pad2): track 0.00 -> 12.5 mm
- net Net-(R29-Pad2): track 0.00 -> 12.5 mm
- net Net-(R28-Pad2): track 0.00 -> 12.5 mm
- net Net-(R23-Pad2): track 0.00 -> 12.5 mm
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- added copper zone on B.Cu, net GND
