File: project_kicad/strange_games.kicad_pcb (KiCad board)
At the start: 2 copper layers, 330 x 247.5 mm, 118 parts, among them J1 Display, M1 Motor_DC, Q1 Si2302A, Q2 Q_Photo, Q3 Si2302A, Q4 Q_Photo, SW1 SW_Push, SW10 SW_Push, SW2 SW_Push, SW3 SW_Push, SW4 SW_Push, SW5 SW_Push, SW6 SW_Push, SW7 SW_Push, SW8 SW_Push, SW9 SW_Push, U1 charge controller, U2 boost converter, U3 LDL1117S33R, U4 ESP32-DEVKIT-V1, U5 TMP112xxDRL, U6 vibrating_sensor, U7 LSM6DS3, U8 MQ-135 gas sensor

Commit message: code changes
Parts:
- moved R1 90.7 mm to (135.7, 174.5), turned to 90 degrees
- moved R2 88.0 mm to (137.7, 174.5), turned to 90 degrees
- moved U7 56.7 mm to (137.2, 178.3)
- moved U5 50.7 mm to (133.9, 177.9)
- moved U4 4.37 mm to (154.7, 159.8)
Routing:
- net +3V3: track 289.2 -> 309.1 mm
Changed lines of the file:
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@@
   )
   (footprint "Package_LGA:LGA-14_3x2.5mm_P0.5mm_LayoutBorder3x4y" (layer "F.Cu")
-    (at 191.097637 160.6)
+    (at 137.202 178.276)
     (descr "LGA, 14 Pin (https://www.st.com/resource/en/datasheet/lsm6ds3tr-c.pdf), generated with kicad-footprint-generator ipc_noLead_generator.py")
     (tags "LGA NoLead")
@@
     (property "ki_keywords" "Accelerometer Gyroscope MEMS")
     (attr smd)
-    (fp_text reference "U7" (at 0 -2.2) (layer "F.SilkS")
+    (fp_text reference "U7" (at 0 2.286) (layer "F.SilkS")
         (effects (font (size 1 1) (thickness 0.15)))
     )
-    (fp_text value "LSM6DS3" (at 0 2.2) (layer "F.Fab")
+    (fp_text value "LSM6DS3" (at 0 2.2) (layer "F.Fab") hide
         (effects (font (size 1 1) (thickness 0.15)))
     )
@@
   )
   (footprint "PCM_4ms_Resistor:R_0805_2012Metric" (layer "F.Cu")
-    (at 223.322 154.004)
+    (at 137.71 174.466 90)
     (descr "Resistor SMD 0805 (2012 Metric), square (rectangular) end terminal, IPC_7351 nominal, (Body size source: https://docs.google.com/spreadsheets/d/1BsfQQcO9C6DZCsRaXUlFlo91Tg2WpOkGARC1WS5S8t0/edit?usp=sharing), generated with kicad-footprint-generator")
     (tags "resistor")
@@
     (property "ki_keywords" "1.2k_0603")
     (attr smd)
-    (fp_text reference "R2" (at 0 -1.65) (layer "F.SilkS")
+    (fp_text reference "R2" (at 2.794 0 90) (layer "F.SilkS")
         (effects (font (size 1 1) (thickness 0.15)))
     )
-    (fp_text value "10k_0805" (at 0 1.65) (layer "F.Fab")
+    (fp_text value "10k_0805" (at 0 1.65 90) (layer "F.Fab") hide
         (effects (font (size 1 1) (thickness 0.15)))
     )
-    (fp_text user "${REFERENCE}" (at 0 0) (layer "F.Fab")
+    (fp_text user "${REFERENCE}" (at 0 0 90) (layer "F.Fab")
         (effects (font (size 0.5 0.5) (thickness 0.08)))
     )
@@
     (fp_line (start 1 0.6) (end -1 0.6)
       (stroke (width 0.1) (type solid)) (layer "F.Fab"))
-    (pad "1" smd roundrect (at -0.9375 0) (size 0.975 1.4) (layers "F.Cu" "F.Paste" "F.Mask") (roundrect_rratio 0.25)
+    (pad "1" smd roundrect (at -0.9375 0 90) (size 0.975 1.4) (layers "F.Cu" "F.Paste" "F.Mask") (roundrect_rratio 0.25)
       (net 40 "SCL") (pintype "passive"))
-    (pad "2" smd roundrect (at 0.9375 0) (size 0.975 1.4) (layers "F.Cu" "F.Paste" "F.Mask") (roundrect_rratio 0.25)
+    (pad "2" smd roundrect (at 0.9375 0 90) (size 0.975 1.4) (layers "F.Cu" "F.Paste" "F.Mask") (roundrect_rratio 0.25)
       (net 21 "+3V3") (pintype "passive"))
     (model "${KISYS3DMOD}/Resistor_SMD.3dshapes/R_0805_2012Metric.wrl"
@@
   )
   (footprint "SnapEDA Library:MODULE_ESP32_DEVKIT_V1" (layer "F.Cu")
-    (at 150.368 159.533)
+    (at 154.728 159.755)
     (property "MANUFACTURER" "DOIT")
     (property "MAXIMUM_PACKAGE_HEIGHT" "6.8 mm")
@@
   )
   (footprint "PCM_4ms_Resistor:R_0805_2012Metric" (layer "F.Cu")
-    (at 223.322 151.054)
+    (at 135.678 174.466 90)
     (descr "Resistor SMD 0805 (2012 Metric), square (rectangular) end terminal, IPC_7351 nominal, (Body size source: https://docs.google.com/spreadsheets/d/1BsfQQcO9C6DZCsRaXUlFlo91Tg2WpOkGARC1WS5S8t0/edit?usp=sharing), generated with kicad-footprint-generator")
     (tags "resistor")
@@
     (property "ki_keywords" "1.2k_0603")
     (attr smd)
-    (fp_text reference "R1" (at 0 -1.65) (layer "F.SilkS")
+    (fp_text reference "R1" (at 2.8725 0 90) (layer "F.SilkS")
         (effects (font (size 1 1) (thickness 0.15)))
     )
-    (fp_text value "10k_0805" (at 0 1.65) (layer "F.Fab")
+    (fp_text value "10k_0805" (at 0 1.65 90) (layer "F.Fab") hide
         (effects (font (size 1 1) (thickness 0.15)))
     )
-    (fp_text user "${REFERENCE}" (at 0 0) (layer "F.Fab")
+    (fp_text user "${REFERENCE}" (at 0 0 90) (layer "F.Fab")
         (effects (font (size 0.5 0.5) (thickness 0.08)))
     )
@@
     (fp_line (start 1 0.6) (end -1 0.6)
       (stroke (width 0.1) (type solid)) (layer "F.Fab"))
-    (pad "1" smd roundrect (at -0.9375 0) (size 0.975 1.4) (layers "F.Cu" "F.Paste" "F.Mask") (roundrect_rratio 0.25)
+    (pad "1" smd roundrect (at -0.9375 0 90) (size 0.975 1.4) (layers "F.Cu" "F.Paste" "F.Mask") (roundrect_rratio 0.25)
       (net 27 "SDA") (pintype "passive"))
-    (pad "2" smd roundrect (at 0.9375 0) (size 0.975 1.4) (layers "F.Cu" "F.Paste" "F.Mask") (roundrect_rratio 0.25)
+    (pad "2" smd roundrect (at 0.9375 0 90) (size 0.975 1.4) (layers "F.Cu" "F.Paste" "F.Mask") (roundrect_rratio 0.25)
       (net 21 "+3V3") (pintype "passive"))
     (model "${KISYS3DMOD}/Resistor_SMD.3dshapes/R_0805_2012Metric.wrl"
@@
   )
   (footprint "Package_TO_SOT_SMD:SOT-563" (layer "F.Cu")
-    (at 181.847637 161.33)
+    (at 133.918418 177.865794)
     (descr "SOT563")
     (tags "SOT-563")
@@
     (property "ki_keywords" "digital temperature sensor i2c smbus two-wire nist")
     (attr smd)
-    (fp_text reference "U5" (at 0 -1.7) (layer "F.SilkS")
+    (fp_text reference "U5" (at 0 1.8495) (layer "F.SilkS")
         (effects (font (size 1 1) (thickness 0.15)))
     )
-    (fp_text value "TMP112xxDRL" (at 0 1.75) (layer "F.Fab")
+    (fp_text value "TMP112xxDRL" (at 0 1.75) (layer "F.Fab") hide
         (effects (font (size 1 1) (thickness 0.15)))
     )
@@
   (segment (start 105.823 135.124) (end 105.823 133.445) (width 0.35) (layer "F.Cu") (net 21))
   (segment (start 104.992066 152.02) (end 86.227 152.02) (width 0.35) (layer "F.Cu") (net 21))
+  (segment (start 137.456 161.0825) (end 137.456 146.812) (width 1) (layer "F.Cu") (net 21))
   (segment (start 85.823 135.124) (end 85.823 133.445) (width 0.35) (layer "F.Cu") (net 21))
   (segment (start 280.292 175.641) (end 274.35 175.641) (width 1) (layer "F.Cu") (net 21))
@@
   (segment (start 65.823 175.124) (end 65.823 173.445) (width 0.35) (layer "F.Cu") (net 21))
   (segment (start 65.823 175.124) (end 65.823 172.850934) (width 0.35) (layer "F.Cu") (net 21))
+  (segment (start 137.456 146.812) (end 140.028 144.24) (width 1) (layer "F.Cu") (net 21))
   (segment (start 66.653934 172.02) (end 85.412066 172.02) (width 0.35) (layer "F.Cu") (net 21))
   (segment (start 104.992066 172.02) (end 105.823 172.850934) (width 0.35) (layer "F.Cu") (net 21))
@@
   (segment (start 105.823 152.850934) (end 104.992066 152.02) (width 0.35) (layer "F.Cu") (net 21))
   (segment (start 85.823 155.124) (end 85.823 153.445) (width 0.35) (layer "F.Cu") (net 21))
+  (segment (start 140.028 144.24) (end 142.028 144.24) (width 1) (layer "F.Cu") (net 21))
   (segment (start 65.823 152.850934) (end 66.653934 152.02) (width 0.35) (layer "F.Cu") (net 21))
   (segment (start 85.823 175.124) (end 85.823 173.445) (width 0.35) (layer "F.Cu") (net 21))
@@
   (segment (start 85.823 132.850934) (end 85.823 133.445) (width 0.35) (layer "F.Cu") (net 21))
   (segment (start 104.553 173.445) (end 88.363 173.445) (width 0.35) (layer "F.Cu") (net 25))
+  (segment (start 135.678 175.482) (end 135.678 175.4035) (width 0.25) (layer "F.Cu") (net 27))
   (segment (start 170.1585 230) (end 168.952 230) (width 1) (layer "F.Cu") (net 28))
   (segment (start 150.1585 210) (end 148.952 210) (width 1) (layer "F.Cu") (net 29))

Commit message: code changes
Parts:
- added C10: C_Generic, PCM_Capacitor_SMD_AKL:C_0402_1005Metric, F.Cu at (338.9, 97.2)
- added C36: C_Generic, PCM_Capacitor_SMD_AKL:C_0402_1005Metric, F.Cu at (338.9, 99.4)
- added C5: C_Generic, PCM_Capacitor_SMD_AKL:C_0402_1005Metric, F.Cu at (338.9, 93.0)
- added C8: C_Generic, PCM_Capacitor_SMD_AKL:C_0402_1005Metric, F.Cu at (338.9, 95.1)
