File: project_kicad/strange_games.kicad_pcb (KiCad board)
At the start: 2 copper layers, 330 x 247.5 mm, 122 parts, among them J1 Display, M1 Motor_DC, Q1 Si2302A, Q2 Q_Photo, Q3 Si2302A, Q4 Q_Photo, SW1 SW_Push, SW10 SW_Push, SW2 SW_Push, SW3 SW_Push, SW4 SW_Push, SW5 SW_Push, SW6 SW_Push, SW7 SW_Push, SW8 SW_Push, SW9 SW_Push, U1 charge controller, U2 boost converter, U3 LDL1117S33R, U4 ESP32-DEVKIT-V1, U5 TMP112xxDRL, U6 vibrating_sensor, U7 LSM6DS3, U8 MQ-135 gas sensor

Commit message: changed 10kR to 330R
Parts:
- removed C50: C_Generic, PCM_Capacitor_SMD_AKL:C_0402_1005Metric
- added C44: C_Generic, PCM_Capacitor_SMD_AKL:C_0402_1005Metric, F.Cu at (352.4, 77.7)
- added R34: 10k_0805, PCM_4ms_Resistor:R_0805_2012Metric, F.Cu at (348.6, 78.1)
- added R35: 10k_0805, PCM_4ms_Resistor:R_0805_2012Metric, F.Cu at (348.6, 81.1)
- added R36: 330_0805, PCM_4ms_Resistor:R_0805_2012Metric, F.Cu at (348.6, 84.0)
- added R37: 330_0805, PCM_4ms_Resistor:R_0805_2012Metric, F.Cu at (348.6, 87.0)
- added R38: 330_0805, PCM_4ms_Resistor:R_0805_2012Metric, F.Cu at (348.6, 89.9)
- added R39: 10k_0805, PCM_4ms_Resistor:R_0805_2012Metric, F.Cu at (348.6, 92.9)
- added R40: 10k_0805, PCM_4ms_Resistor:R_0805_2012Metric, F.Cu at (348.6, 95.8)
- added R41: 10k_0805, PCM_4ms_Resistor:R_0805_2012Metric, F.Cu at (348.6, 98.8)
- C10, C31: footprint PCM_Capacitor_SMD_AKL:C_0402_1005Metric -> PCM_Capacitor_SMD_AKL:C_0805_2012Metric
- C12, C33: footprint PCM_Capacitor_SMD_AKL:C_0805_2012Metric -> PCM_Capacitor_SMD_AKL:C_0402_1005Metric
- R14, R16, R20, R21, R22, R29, R30, R31: value 10k_0805 -> 330_0805
- R3: value 10k_0805 -> 100_0805
- moved R11 142.6 mm to (306.7, 83.3)
- moved R8 142.6 mm to (306.7, 77.4)
- moved C22 142.6 mm to (310.5, 74.0)
- moved C23 142.6 mm to (310.5, 76.1)
- moved C48 142.6 mm to (310.5, 88.9)
- moved R10 142.6 mm to (306.7, 80.3)
- moved R20 142.6 mm to (306.7, 86.2)
- moved R27 142.6 mm to (306.7, 89.2)
- moved R7 142.6 mm to (306.7, 74.4)
- moved C41 142.6 mm to (306.9, 71.4)
- moved C31 71.3 mm to (136.2, 186.1)
Connections:
- C10 pad 1: +3V3 -> GND
- C10 pad 2: GND -> +12V
- C11 pad 2: +12V -> +3V3
- C12 pad 1: GND -> Net-(J1-CAP5+)
- C12 pad 2: +3V3 -> Net-(J1-CAP1-)
- C13 pad 1: Net-(J1-CAP5+) -> Net-(J1-CAP2+)
- C13 pad 2: Net-(J1-CAP1-) -> Net-(J1-CAP2-)
- C14 pad 1: Net-(J1-CAP2+) -> Net-(J1-CAP4+)
- C15 pad 1: Net-(J1-CAP4+) -> +3V3
- C15 pad 2: Net-(J1-CAP2-) -> Net-(J1-V3)
- C16 pad 2: Net-(J1-V3) -> Net-(J1-V1)
- C17 pad 1: +3V3 -> Net-(J1-Vout)
- C17 pad 2: Net-(J1-V1) -> GND
- C18 pad 1: Net-(J1-Vout) -> Net-(J1-CAP3+)
- C18 pad 2: GND -> Net-(J1-CAP1-)
- C19 pad 1: Net-(J1-CAP3+) -> Net-(J1-CAP1+)
- C20 pad 1: Net-(J1-CAP1+) -> +3V3
- C20 pad 2: Net-(J1-CAP1-) -> Net-(J1-V4)
- C21 pad 2: Net-(J1-V4) -> Net-(J1-V2)
- C22 pad 2: Net-(J1-V2) -> Net-(J1-V0)
- C23 pad 1: +3V3 -> B1
- C23 pad 2: Net-(J1-V0) -> +3V3
- C24 pad 1: B1 -> B2
- C25 pad 1: B2 -> B3
- C26 pad 1: B3 -> B4
- C27 pad 1: B4 -> B5
- C28 pad 1: B5 -> B6
- C29 pad 1: B6 -> GND
- C30 pad 1: GND -> +3V3
- C30 pad 2: +3V3 -> GND
- C31 pad 1: +3V3 -> GND
- C31 pad 2: GND -> +3V3
- C33 pad 1: GND -> +3V3
- C33 pad 2: +3V3 -> GND
- C36 pad 1: +3V3 -> B7
- C36 pad 2: GND -> +3V3
- C37 pad 1: B7 -> B8
- C38 pad 1: B8 -> B9
- C39 pad 1: B9 -> GND
- C42 pad 1: GND -> +3V3
- C42 pad 2: +3V3 -> GND
- C43 pad 1: +3V3 -> GND
- C43 pad 2: GND -> +3V3
- C48 pad 1: GND -> +3V3
- C48 pad 2: +3V3 -> GND
- C49 pad 1: +3V3 -> GND
- C49 pad 2: GND -> +3V3
- C8 pad 1: +3V3 -> GND
- C8 pad 2: GND -> +3V3
- C9 pad 1: GND -> +3V3
- C9 pad 2: +3V3 -> GND
- D11 pad 4: Net-(D10-DO) -> Net-(D11-DI)
- D12 pad 4: Net-(D11-DO) -> Net-(D12-DI)
- D13 pad 4: Net-(D12-DO) -> Net-(D10-DO)
- D6 pad 4: Net-(D5-DO) -> Net-(D11-DO)
- D7 pad 1: Net-(D7-DO) -> Net-(D10-DI)
- D7 pad 4: Net-(D6-DO) -> Net-(D12-DO)
- D8 pad 1: Net-(D8-DO) -> Net-(D11-DI)
- D8 pad 4: Net-(D7-DO) -> Net-(D5-DO)
- D9 pad 1: Net-(D10-DI) -> Net-(D12-DI)
- D9 pad 4: Net-(D8-DO) -> Net-(D6-DO)
- J1 pad 24: unconnected-(J1-D5-Pad24) -> Net-(J1-D5)
- J1 pad 25: unconnected-(J1-D4-Pad25) -> Net-(J1-D4)
- J1 pad 26: unconnected-(J1-D3-Pad26) -> Net-(J1-D3)
- J1 pad 27: unconnected-(J1-D2-Pad27) -> Net-(J1-D2)
- J1 pad 28: unconnected-(J1-D1-Pad28) -> Net-(J1-D1)
- J1 pad 29: unconnected-(J1-D0-Pad29) -> Net-(J1-D0)
- R10 pad 1: Net-(Q3-G) -> Net-(J1-D2)
- R10 pad 2: vibrating_motor -> GND
- R11 pad 1: GND -> Net-(J1-D3)
- R11 pad 2: Net-(Q3-G) -> GND
- R12 pad 1: GND -> Net-(J1-D4)
- R12 pad 2: photo_1 -> GND
- R13 pad 1: B1 -> Net-(J1-D5)
- R13 pad 2: Net-(R13-Pad2) -> GND
- R14 pad 1: B2 -> Net-(Q1-G)
- R14 pad 2: Net-(R14-Pad2) -> open_box
- R15 pad 1: B3 -> GND
- R15 pad 2: Net-(R15-Pad2) -> Net-(Q1-G)
- R16 pad 1: GND -> Net-(Q3-G)
- R16 pad 2: photo_2 -> vibrating_motor
- R17 pad 2: Net-(R13-Pad2) -> Net-(Q3-G)
- R18 pad 2: Net-(R14-Pad2) -> photo_1
- R19 pad 2: Net-(R15-Pad2) -> photo_2
- R20 pad 1: GND -> Net-(R20-Pad1)
- R20 pad 2: vibrating_signal -> B1
- R21 pad 1: B4 -> Net-(R21-Pad1)
- R21 pad 2: Net-(R21-Pad2) -> B2
- R22 pad 1: B5 -> Net-(R22-Pad1)
- R22 pad 2: Net-(R22-Pad2) -> B3
- R23 pad 1: B6 -> GND
- R23 pad 2: Net-(R23-Pad2) -> Net-(R20-Pad1)
- R24 pad 2: Net-(R21-Pad2) -> Net-(R21-Pad1)
- R25 pad 2: Net-(R22-Pad2) -> Net-(R22-Pad1)
- R26 pad 1: GND -> Net-(U7-SDX)
- R26 pad 2: Net-(R23-Pad2) -> GND
- R27 pad 1: GND -> Net-(U7-SCX)
- R27 pad 2: gas_signal -> GND
- R28 pad 1: B7 -> GND
- R28 pad 2: Net-(R28-Pad2) -> vibrating_signal
- R29 pad 1: B8 -> Net-(R29-Pad1)
- R29 pad 2: Net-(R29-Pad2) -> B4
- R3 pad 1: B10 -> Net-(R3-Pad1)
- R3 pad 2: Net-(R3-Pad2) -> B10
- R30 pad 1: B9 -> Net-(R30-Pad1)
- R30 pad 2: Net-(R30-Pad2) -> B5
- R31 pad 1: unconnected-(R31-Pad1) -> Net-(R31-Pad1)
- R31 pad 2: Net-(R28-Pad2) -> B6
- R32 pad 2: Net-(R29-Pad2) -> Net-(R29-Pad1)
- R33 pad 2: Net-(R30-Pad2) -> Net-(R30-Pad1)
- R4 pad 2: Net-(R3-Pad2) -> Net-(R3-Pad1)
- R8 pad 1: Net-(Q1-G) -> Net-(J1-D0)
- R8 pad 2: open_box -> GND
- R9 pad 1: GND -> Net-(J1-D1)
- R9 pad 2: Net-(Q1-G) -> GND
- SW1 pad 2: Net-(R3-Pad2) -> Net-(R3-Pad1)
- SW10 pad 2: Net-(R30-Pad2) -> Net-(R38-Pad1)
- SW2 pad 2: Net-(R13-Pad2) -> Net-(R20-Pad1)
- SW3 pad 2: Net-(R14-Pad2) -> Net-(R21-Pad1)
- SW4 pad 2: Net-(R15-Pad2) -> Net-(R22-Pad1)
- SW5 pad 2: Net-(R21-Pad2) -> Net-(R29-Pad1)
- SW6 pad 2: Net-(R22-Pad2) -> Net-(R30-Pad1)
- SW7 pad 2: Net-(R23-Pad2) -> Net-(R31-Pad1)
- SW8 pad 2: Net-(R28-Pad2) -> Net-(R36-Pad1)
- SW9 pad 2: Net-(R29-Pad2) -> Net-(R37-Pad1)
- U7 pad 2: unconnected-(U7-SDX-Pad2) -> Net-(U7-SDX)
- U7 pad 3: unconnected-(U7-SCX-Pad3) -> Net-(U7-SCX)
Routing:
- net (no net): track 0.00 -> 104.4 mm
- net Net-(D7-DO): track 54.4 -> 0.00 mm
- net +3V3: track 309.1 -> 289.2 mm
- net Net-(D8-DO): track 16.2 -> 0.00 mm
- net Net-(D6-DO): track 16.2 -> 32.4 mm
- net GND: track 0.00 -> 14.9 mm
- net B2: track 1.21 -> 14.9 mm
- net Net-(R30-Pad2): track 12.5 -> 0.00 mm
- net Net-(R3-Pad2): track 12.5 -> 0.00 mm
- net Net-(R3-Pad1): track 0.00 -> 12.5 mm
- net Net-(R29-Pad2): track 12.5 -> 0.00 mm
- net Net-(R28-Pad2): track 12.5 -> 0.00 mm
- net Net-(R23-Pad2): track 12.5 -> 0.00 mm
- net Net-(R22-Pad2): track 12.5 -> 0.00 mm
- net Net-(R21-Pad2): track 12.5 -> 0.00 mm
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
Commit message: pcb changes
Parts:
- U8: footprint Connector_PinHeader_1.27mm:PinHeader_1x04_P1.27mm_Vertical -> Connector_PinHeader_2.54mm:PinHeader_1x04_P2.54mm_Vertical
- moved U6 146.4 mm to (200.0, 155.0)
- moved U2 100.5 mm to (155.0, 187.5), turned to 90 degrees
- moved C19 93.5 mm to (184.1, 165.0)
- moved C21 93.5 mm to (184.1, 167.3)
- moved D2 93.5 mm to (183.6, 162.7)
- moved U3 93.5 mm to (185.4, 157.6)
- moved C4 93.5 mm to (179.1, 162.7)
- moved D3 69.0 mm to (278.9, 119.2)
- moved D4 69.0 mm to (278.9, 122.5)
- moved R9 69.0 mm to (266.4, 137.5)
- moved R16 69.0 mm to (260.6, 118.2)
- moved C31 65.9 mm to (163.5, 126.2), turned to 90 degrees
- moved L1 62.9 mm to (279.2, 156.4)
- moved M1 62.9 mm to (279.2, 147.3)
- moved Q2 62.9 mm to (272.1, 150.3)
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
Commit message: remastered display pins in the kicad scheme
Parts:
- added C50: C_Generic, PCM_Capacitor_SMD_AKL:C_0402_1005Metric, F.Cu at (143.7, 47.8)
- added R42: 10k_0805, PCM_4ms_Resistor:R_0805_2012Metric, F.Cu at (139.9, 48.2)
- added SW11: SW_Push, Button_Switch_THT:SW_PUSH-12mm, F.Cu at (140.0, 37.5)
- C10, C11, C2, C31, C41, C7: footprint PCM_Capacitor_SMD_AKL:C_0805_2012Metric -> PCM_Capacitor_SMD_AKL:C_0402_1005Metric
- C16, C17, C32, C42, C5, C8: footprint PCM_Capacitor_SMD_AKL:C_0402_1005Metric -> PCM_Capacitor_SMD_AKL:C_0805_2012Metric
- R14, R16, R20, R29, R36: value 330_0805 -> 10k_0805
- R15, R17, R23, R32, R39, R4: value 10k_0805 -> 330_0805
- R3: value 100_0805 -> 330_0805
Connections:
- C10 pad 2: +12V -> +3V3
- C11 pad 1: GND -> +3V3
- C11 pad 2: +3V3 -> Net-(J1-V4)
- C12 pad 1: Net-(J1-CAP5+) -> +3V3
- C12 pad 2: Net-(J1-CAP1-) -> Net-(J1-V2)
- C13 pad 1: Net-(J1-CAP2+) -> +3V3
- C13 pad 2: Net-(J1-CAP2-) -> Net-(J1-V0)
- C14 pad 1: Net-(J1-CAP4+) -> +3V3
- C14 pad 2: Net-(J1-CAP2-) -> Net-(J1-V3)
- C15 pad 2: Net-(J1-V3) -> Net-(J1-V1)
- C16 pad 1: +3V3 -> GND
- C16 pad 2: Net-(J1-V1) -> +12V
- C17 pad 1: Net-(J1-Vout) -> GND
- C17 pad 2: GND -> +3V3
- C18 pad 1: Net-(J1-CAP3+) -> Net-(J1-CAP5+)
- C19 pad 1: Net-(J1-CAP1+) -> Net-(J1-CAP2+)
- C19 pad 2: Net-(J1-CAP1-) -> Net-(J1-CAP2-)
- C2 pad 1: GND -> +3V3
- C2 pad 2: +3V3 -> GND
- C20 pad 1: +3V3 -> Net-(J1-CAP4+)
- C20 pad 2: Net-(J1-V4) -> Net-(J1-CAP2-)
- C21 pad 1: +3V3 -> Net-(J1-CAP3+)
- C21 pad 2: Net-(J1-V2) -> Net-(J1-CAP1-)
- C22 pad 1: +3V3 -> Net-(J1-CAP1+)
- C22 pad 2: Net-(J1-V0) -> Net-(J1-CAP1-)
- C23 pad 1: B1 -> Net-(J1-Vout)
- C23 pad 2: +3V3 -> GND
- C24 pad 1: B2 -> B1
- C25 pad 1: B3 -> B2
- C26 pad 1: B4 -> B3
- C27 pad 1: B5 -> B4
- C28 pad 1: B6 -> B5
- C29 pad 1: GND -> B6
- C30 pad 1: +3V3 -> GND
- C30 pad 2: GND -> +3V3
- C31 pad 1: GND -> +3V3
- C31 pad 2: +3V3 -> GND
- C33 pad 1: +3V3 -> GND
- C33 pad 2: GND -> +3V3
- C35 pad 1: GND -> +3V3
- C35 pad 2: +3V3 -> GND
- C36 pad 1: B7 -> GND
- C37 pad 1: B8 -> B7
- C38 pad 1: B9 -> B8
- C39 pad 1: GND -> B9
- C42 pad 1: +3V3 -> GND
- C42 pad 2: GND -> +3V3
- C43 pad 1: GND -> +3V3
- C43 pad 2: +3V3 -> GND
- C44 pad 1: +3V3 -> GND
- C44 pad 2: GND -> +3V3
- C45 pad 1: GND -> +3V3
- C45 pad 2: +3V3 -> GND
- C48 pad 1: +3V3 -> GND
- C48 pad 2: GND -> +3V3
- C49 pad 1: GND -> +3V3
- C49 pad 2: +3V3 -> GND
- C5 pad 1: +3V3 -> GND
- C5 pad 2: GND -> +3V3
- C7 pad 1: GND -> B11
- J1 pad 22: SDA -> MOSI
- J1 pad 30: RD_display -> Net-(J1-/RD(E))
- J1 pad 31: WR_display -> Net-(J1-/WR(RW))
- J1 pad 33: GND -> +3V3
- R10 pad 1: Net-(J1-D2) -> Net-(J1-D1)
- R10 pad 2: GND -> +3V3
- R11 pad 1: Net-(J1-D3) -> Net-(J1-D2)
- R11 pad 2: GND -> +3V3
- R12 pad 1: Net-(J1-D4) -> Net-(J1-D3)
- R12 pad 2: GND -> +3V3
- R13 pad 1: Net-(J1-D5) -> Net-(J1-D4)
- R13 pad 2: GND -> +3V3
- R14 pad 1: Net-(Q1-G) -> Net-(J1-D5)
- R14 pad 2: open_box -> +3V3
- R15 pad 1: GND -> Net-(Q1-G)
- R15 pad 2: Net-(Q1-G) -> open_box
- R16 pad 1: Net-(Q3-G) -> GND
- R16 pad 2: vibrating_motor -> Net-(Q1-G)
- R17 pad 1: GND -> Net-(Q3-G)
- R17 pad 2: Net-(Q3-G) -> vibrating_motor
- R18 pad 2: photo_1 -> Net-(Q3-G)
- R19 pad 2: photo_2 -> photo_1
- R20 pad 1: Net-(R20-Pad1) -> GND
- R20 pad 2: B1 -> photo_2
- R21 pad 2: B2 -> B1
- R22 pad 2: B3 -> B2
- R23 pad 1: GND -> Net-(R23-Pad1)
- R23 pad 2: Net-(R20-Pad1) -> B3
- R26 pad 1: Net-(U7-SDX) -> GND
- R26 pad 2: GND -> Net-(R23-Pad1)
- R27 pad 1: Net-(U7-SCX) -> Net-(U7-SDX)
- R28 pad 1: GND -> Net-(U7-SCX)
- R28 pad 2: vibrating_signal -> GND
- R29 pad 1: Net-(R29-Pad1) -> GND
- R29 pad 2: B4 -> vibrating_signal
- R30 pad 2: B5 -> B4
- R31 pad 2: B6 -> B5
- R32 pad 1: GND -> Net-(R32-Pad1)
- R32 pad 2: Net-(R29-Pad1) -> B6
- R35 pad 2: gas_signal -> Net-(R32-Pad1)
- R36 pad 1: Net-(R36-Pad1) -> GND
- R36 pad 2: B7 -> gas_signal
- R37 pad 2: B8 -> B7
- R38 pad 2: B9 -> B8
- R39 pad 1: unconnected-(R39-Pad1) -> Net-(R39-Pad1)
- R39 pad 2: Net-(R36-Pad1) -> B9
- R4 pad 1: GND -> Net-(R4-Pad1)
- R4 pad 2: Net-(R3-Pad1) -> B11
- R40 pad 1: GND -> unconnected-(R40-Pad1)
- R5 pad 1: A0_display -> GND
- R5 pad 2: +3V3 -> Net-(R3-Pad1)
- R6 pad 1: WR_display -> GND
- R6 pad 2: +3V3 -> Net-(R4-Pad1)
- R7 pad 1: RD_display -> Net-(J1-/WR(RW))
- R8 pad 1: Net-(J1-D0) -> Net-(J1-/RD(E))
- R8 pad 2: GND -> +3V3
- R9 pad 1: Net-(J1-D1) -> Net-(J1-D0)
- R9 pad 2: GND -> +3V3
- SW2 pad 2: Net-(R20-Pad1) -> Net-(R4-Pad1)
- SW5 pad 2: Net-(R29-Pad1) -> Net-(R23-Pad1)
- SW8 pad 2: Net-(R36-Pad1) -> Net-(R32-Pad1)
- U4 pad 10: RD_display -> photo_1
- U4 pad 26: gas_signal -> CLK
- U4 pad 27: photo_2 -> B11
- U4 pad 28: photo_1 -> MOSI
- U4 pad 9: WR_display -> photo_2
Routing:
- net GND: track 14.9 -> 13.7 mm
- net B6: track 1.21 -> 2.41 mm

Commit message: pcb updates
Parts:
- removed C8: C_Generic, PCM_Capacitor_SMD_AKL:C_0805_2012Metric
- removed C9: C_Generic, PCM_Capacitor_SMD_AKL:C_0402_1005Metric
- removed the R34 at (348.6, 78.1)
- removed the R35 at (348.6, 81.1)
- removed the R37 at (348.6, 87.0)
- removed the R38 at (348.6, 89.9)
- removed the R39 at (348.6, 92.9)
- removed the R40 at (348.6, 95.8)
- removed the R41 at (348.6, 98.8)
- removed the R42 at (139.9, 48.2)
- removed SW1: SW_Push, Button_Switch_THT:SW_PUSH-12mm
- removed the SW11 at (140.0, 37.5)
- added R13: 10k_0805, PCM_4ms_Resistor:R_0805_2012Metric, F.Cu at (187.9, 113.5)
- added R14: 10k_0805, PCM_4ms_Resistor:R_0805_2012Metric, F.Cu at (186.0, 113.5)
- added R15: 330_0805, PCM_4ms_Resistor:R_0805_2012Metric, F.Cu at (272.1, 220.2)
- added R17: 330_0805, PCM_4ms_Resistor:R_0805_2012Metric, F.Cu at (270.8, 206.8)
- added R18: 10k_0805, PCM_4ms_Resistor:R_0805_2012Metric, F.Cu at (268.5, 210.3)
- added R26: 10k_0805, PCM_4ms_Resistor:R_0805_2012Metric, F.Cu at (191.1, 212.5)
- added R28: 330_0805, PCM_4ms_Resistor:R_0805_2012Metric, F.Cu at (251.8, 216.8)
- added R29: 10k_0805, PCM_4ms_Resistor:R_0805_2012Metric, F.Cu at (298.1, 203.0)
- C10, C19, C20, C45, R1, R2: moved to B.Cu
- C2: footprint PCM_Capacitor_SMD_AKL:C_0402_1005Metric -> PCM_Capacitor_SMD_AKL:C_0805_2012Metric
- C42: footprint PCM_Capacitor_SMD_AKL:C_0805_2012Metric -> PCM_Capacitor_SMD_AKL:C_0402_1005Metric; moved to B.Cu
- L1: value L_Iron -> L_iron
- R21: renamed from R13; value 10k_0805 -> 330_0805
- R22: renamed from R17; value 330_0805 -> 10k_0805
- R23: renamed from R14; value 10k_0805 -> 330_0805
- R27: value 10k_0805 -> 330_0805
- R37: renamed from R28; value 10k_0805 -> 330_0805
- R38: renamed from R31; value 330_0805 -> 10k_0805
- R39: renamed from R29; value 10k_0805 -> 330_0805
- R40: renamed from R32; value 330_0805 -> 10k_0805
- RV1: value TRIM -> R_Potentiometer
- moved C44 193.0 mm to (167.9, 134.4), turned to 180 degrees
- moved C17 185.8 mm to (50.3, 242.3), turned to 180 degrees
- moved D1 182.5 mm to (74.4, 227.7)
- moved C4 164.9 mm to (37.5, 247.3)
- moved U3 164.9 mm to (43.9, 242.2)
- moved D2 164.9 mm to (42.1, 247.3)
- moved C5 159.9 mm to (236.5, 215.8), turned to -90 degrees
- moved C16 159.5 mm to (72.0, 224.8)
- moved C41 153.1 mm to (165.9, 131.0), turned to -90 degrees
- moved C10 146.6 mm to (194.3, 121.8), turned to 90 degrees
- moved R27 143.8 mm to (238.5, 215.8), turned to 90 degrees
- moved R36 142.3 mm to (307.3, 220.2), turned to 180 degrees
- moved R20 140.9 mm to (253.8, 216.8), turned to 90 degrees
- moved C22 132.7 mm to (184.8, 116.7), turned to 90 degrees
- moved C23 129.2 mm to (187.8, 116.7), turned to 90 degrees
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- renumbered R18 to R24, R15 to R25, R21 to R30, R24 to R31, R22 to R32, R25 to R33, R23 to R34, R26 to R35, R30 to R41, R33 to R42, SW9 to SW10, SW10 to SW11, SW2 to SW3, SW3 to SW4, SW4 to SW5, SW5 to SW6, SW6 to SW7, SW7 to SW8, SW8 to SW9
Connections:
- C2 pad 1: +3V3 -> GND
- C2 pad 2: GND -> Net-(C2-Pad2)
- C42 pad 1: GND -> +3V3
- C42 pad 2: +3V3 -> GND
- C5 pad 2: +3V3 -> Net-(C5-Pad2)
- D11 pad 4: Net-(D11-DI) -> Net-(D10-DO)
- D12 pad 4: Net-(D12-DI) -> Net-(D11-DO)
- D13 pad 4: Net-(D10-DO) -> Net-(D12-DO)
- D3 pad 1: +12V -> +3V3
- D3 pad 2: Net-(D3-A) -> Net-(D4-A)
- D6 pad 4: Net-(D11-DO) -> Net-(D5-DO)
- D7 pad 1: Net-(D10-DI) -> Net-(D7-DO)
- D7 pad 4: Net-(D12-DO) -> Net-(D6-DO)
- D8 pad 1: Net-(D11-DI) -> Net-(D8-DO)
- D8 pad 4: Net-(D5-DO) -> Net-(D7-DO)
- D9 pad 1: Net-(D12-DI) -> Net-(D10-DI)
- D9 pad 4: Net-(D6-DO) -> Net-(D8-DO)
- L1 pad 1: +12V -> +3V3
- L1 pad 2: Net-(D3-A) -> Net-(D4-A)
- Q1 pad 1: Net-(Q1-G) -> Net-(Q3-G)
- Q1 pad 3: Net-(D3-A) -> Net-(D4-A)
- R16 pad 2: Net-(Q1-G) -> Net-(Q3-G)
- R21 pad 1: Net-(J1-D4) -> Net-(R21-Pad1)
- R21 pad 2: +3V3 -> B1
- R22 pad 1: Net-(Q3-G) -> GND
- R22 pad 2: vibrating_motor -> Net-(R21-Pad1)
- R23 pad 1: Net-(J1-D5) -> Net-(R23-Pad1)
- R23 pad 2: +3V3 -> B2
- R24 pad 2: Net-(Q3-G) -> Net-(R23-Pad1)
- R25 pad 1: Net-(Q1-G) -> Net-(R25-Pad1)
- R25 pad 2: open_box -> B3
- R27 pad 1: Net-(U7-SDX) -> Net-(C5-Pad2)
- R27 pad 2: GND -> photo_1
- R30 pad 1: Net-(R21-Pad1) -> Net-(R30-Pad1)
- R30 pad 2: B1 -> B4
- R31 pad 2: Net-(R21-Pad1) -> Net-(R30-Pad1)
- R32 pad 1: Net-(R22-Pad1) -> Net-(R32-Pad1)
- R32 pad 2: B2 -> B5
- R33 pad 2: Net-(R22-Pad1) -> Net-(R32-Pad1)
- R34 pad 1: Net-(R23-Pad1) -> Net-(R34-Pad1)
- R34 pad 2: B3 -> B6
- R35 pad 2: Net-(R23-Pad1) -> Net-(R34-Pad1)
- R37 pad 1: Net-(U7-SCX) -> Net-(R37-Pad1)
- R37 pad 2: GND -> B7
- R38 pad 1: Net-(R31-Pad1) -> GND
- R38 pad 2: B5 -> Net-(R37-Pad1)
- R39 pad 1: GND -> Net-(R39-Pad1)
- R39 pad 2: vibrating_signal -> B8
- R40 pad 1: Net-(R32-Pad1) -> GND
- R40 pad 2: B6 -> Net-(R39-Pad1)
- R41 pad 1: Net-(R30-Pad1) -> Net-(R41-Pad1)
- R41 pad 2: B4 -> B9
- R42 pad 2: Net-(R30-Pad1) -> Net-(R41-Pad1)
- RV1 pad 1: +3V3 -> Net-(J1-V0)
- SW10 pad 2: Net-(R37-Pad1) -> Net-(R39-Pad1)
- SW11 pad 2: Net-(R38-Pad1) -> Net-(R41-Pad1)
- SW3 pad 2: Net-(R4-Pad1) -> Net-(R21-Pad1)
- SW4 pad 2: Net-(R21-Pad1) -> Net-(R23-Pad1)
- SW5 pad 2: Net-(R22-Pad1) -> Net-(R25-Pad1)
- SW6 pad 2: Net-(R23-Pad1) -> Net-(R30-Pad1)
- SW7 pad 2: Net-(R30-Pad1) -> Net-(R32-Pad1)
- SW8 pad 2: Net-(R31-Pad1) -> Net-(R34-Pad1)
- SW9 pad 2: Net-(R32-Pad1) -> Net-(R37-Pad1)
- U4 pad 10: photo_1 -> INT1
- U4 pad 12: INT2 -> photo_1
- U4 pad 13: INT1 -> B6
- U4 pad 15: B6 -> INT2
- U7 pad 2: Net-(U7-SDX) -> GND
- U7 pad 3: Net-(U7-SCX) -> GND
Routing:
- net +3V3: track 289.2 -> 68.5 mm, vias 0 -> 5
- net (no net): track 104.4 -> 0.00 mm
- net Net-(D10-DO): track 53.2 -> 18.6 mm
- net VDC: track 4.99 -> 32.1 mm
- net GND: track 13.7 -> 35.9 mm, vias 0 -> 22
- net Net-(D7-DO): track 0.00 -> 21.5 mm
- net Net-(D8-DO): track 0.00 -> 16.2 mm
- net Net-(D6-DO): track 32.4 -> 16.2 mm
- net B2: track 14.9 -> 1.21 mm
- net Net-(D4-A): track 0.00 -> 13.7 mm
- net Net-(J1-V0): track 0.00 -> 12.6 mm
- net Net-(R41-Pad1): track 0.00 -> 12.5 mm
- net Net-(R39-Pad1): track 0.00 -> 12.5 mm
- net Net-(R37-Pad1): track 0.00 -> 12.5 mm
- net Net-(R34-Pad1): track 0.00 -> 12.5 mm
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- added copper zone on F.Cu, net +3V3
- added copper zone on F.Cu, net GND
