File: ProjectKicad/strange_games.kicad_pcb (KiCad board)
At the start: 2 copper layers, 166 x 166 mm, 216 parts, among them J1 Display, M1 Motor_DC, Q1 Si2302A, Q3 Si2302A, Q4 Q_Photo, SW1 SW_Push, SW10 SW_Push, SW11 SW_Push, SW2 SW_Push, SW3 SW_Push, SW4 SW_Push, SW5 SW_Push, SW6 SW_Push, SW7 SW_Push, SW8 SW_Push, SW9 SW_Push, U1 charge controller, U2 boost converter, U3 LDL1117S33R, U4 ESP32-DEVKIT-V1, U5 TMP112xxDRL, U6 vibrating_sensor, U7 LSM6DS3, U8 MQ-135 gas sensor

Commit message: trying to interop
Connections:
- U4 pad 12: Alert -> unconnected-(U4-RX0-Pad12)
- U4 pad 13: Luminodiodes -> unconnected-(U4-TX0-Pad13)
- U4 pad 19: Door -> B2
- U4 pad 20: VibrationMotor -> B1
- U4 pad 21: B2 -> Door
- U4 pad 22: B1 -> VibrationMotor
- U4 pad 9: unconnected-(U4-D18-Pad9) -> Luminodiodes
Routing:
- net GND: track 136.7 -> 166.5 mm, vias 34 -> 27
- net Luminodiodes: track 60.7 -> 44.3 mm
- net VibrationMotor: track 43.3 -> 37.4 mm
- net Door: track 51.2 -> 45.9 mm
- net B2: track 156.9 -> 158.6 mm
- net B1: track 134.2 -> 135.0 mm
