File: ProjectKicad/strange_games.kicad_sch (KiCad schematic)
At the start: 93 parts, among them J1 Display, M1 Motor_DC, Q1 Si2302A, Q3 Si2302A, Q4 Q_Photo, SW1 SW_Push, SW10 SW_Push, SW11 SW_Push, SW2 SW_Push, SW3 SW_Push, SW4 SW_Push, SW5 SW_Push, SW6 SW_Push, SW7 SW_Push, SW8 SW_Push, SW9 SW_Push, U1 charge controller, U2 boost converter, U3 LDL1117S33R, U4 ESP32-DEVKIT-V1, U5 TMP112xxDRL, U6 vibrating_sensor, U7 LSM6DS3, U8 MQ-135 gas sensor

Commit message: trying to interop
Connections:
- net Alert: no longer U4.12 (RX0)
- net B1: now also U4.20 (D35); no longer U4.22 (D33)
- net B2: now also U4.19 (D34); no longer U4.21 (D32)
- net Door: now also U4.21 (D32); no longer U4.19 (D34)
- net Luminodiodes: now also U4.9 (D18); no longer U4.13 (TX0)
- net VibrationMotor: now also U4.22 (D33); no longer U4.20 (D35)
- no-connect marks 7 -> 8
Other:
- moved on the sheet: R1, R2
